File: pcb/prova/prova.kicad_pcb (KiCad board)
At the start: 2 copper layers, 30 x 29 mm, 6 parts, among them J1 Conn_01x04, U1 SN74AHCT125N

Commit message: PCB, F1: regole del DRC in una fonte unica (pcb/regole/hex2.kicad_dru) copiata nei progetti da regole.py; prova con 5V_REG da 1,5 e caso di controllo delle larghezze
Parts:
- turned JP1 to 90 degrees
- renumbered U1 to U3
Connections:
- net /5V renamed /5V_REG
Routing:
- net /5V_REG: track 27.1 -> 25.5 mm
- net /OE1: track 5.44 -> 4.26 mm
Changed lines of the file:
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@@
 			(layers "*.Cu" "*.Mask")
 			(remove_unused_layers no)
-			(net "/5V")
+			(net "/5V_REG")
 		)
 		(pad "2" thru_hole circle
@@
 	(footprint "hex2:SolderJumper-3_P1.3mm_Bridged12_RoundedPad1.0x1.5mm"
 		(layer "F.Cu")
-		(at 9.6 5.5)
+		(at 9.6 5.5 90)
 		(descr "SMD Solder 3-pad Jumper, 1x1.5mm rounded Pads, 0.3mm gap, pads 1-2 bridged with 1 copper strip")
 		(tags "net tie solder jumper bridged")
 		(property "Reference" "JP1"
-			(at 0 -1.8 0)
+			(at 0 -1.8 90)
 			(layer "F.SilkS")
 			(effects
@@
 		)
 		(property "Value" "OE"
-			(at 0 1.9 0)
+			(at 0 1.9 90)
 			(layer "F.Fab")
 			(effects
@@
 		)
 		(property "Datasheet" ""
-			(at 0 0 0)
+			(at 0 0 90)
 			(unlocked yes)
 			(layer "F.Fab")
@@
 		)
 		(property "Description" "3-pole Solder Jumper, pins 1+2 closed/bridged"
-			(at 0 0 0)
+			(at 0 0 90)
 			(unlocked yes)
 			(layer "F.Fab")
@@
 		)
 		(fp_line
+			(start -1.4 -1)
+			(end 1.4 -1)
+			(stroke
+				(width 0.12)
+				(type solid)
+			)
+			(layer "F.SilkS")
+		)
+		(fp_line
+			(start 2.05 -0.3)
+			(end 2.05 0.3)
+			(stroke
+				(width 0.12)
+				(type solid)
+			)
+			(layer "F.SilkS")
+		)
+		(fp_line
 			(start -2.05 0.3)
 			(end -2.05 -0.3)
@@
 		)
 		(fp_line
+			(start 1.4 1)
+			(end -1.4 1)
+			(stroke
+				(width 0.12)
+				(type solid)
+			)
+			(layer "F.SilkS")
+		)
+		(fp_line
+			(start -1.2 1.2)
+			(end -0.9 1.5)
+			(stroke
+				(width 0.12)
+				(type solid)
+			)
+			(layer "F.SilkS")
+		)
+		(fp_line
+			(start -1.2 1.2)
+			(end -1.5 1.5)
+			(stroke
+				(width 0.12)
+				(type solid)
+			)
+			(layer "F.SilkS")
+		)
+		(fp_line
 			(start -1.5 1.5)
 			(end -0.9 1.5)
@@
 			(layer "F.SilkS")
 		)
-		(fp_line
-			(start -1.4 -1)
-			(end 1.4 -1)
-			(stroke
-				(width 0.12)
-				(type solid)
-			)
-			(layer "F.SilkS")
-		)
-		(fp_line
-			(start -1.2 1.2)
-			(end -1.5 1.5)
-			(stroke
-				(width 0.12)
-				(type solid)
-			)
-			(layer "F.SilkS")
-		)
-		(fp_line
-			(start -1.2 1.2)
-			(end -0.9 1.5)
-			(stroke
-				(width 0.12)
-				(type solid)
-			)
-			(layer "F.SilkS")
-		)
-		(fp_line
-			(start 1.4 1)
-			(end -1.4 1)
-			(stroke
-				(width 0.12)
-				(type solid)
-			)
-			(layer "F.SilkS")
-		)
-		(fp_line
-			(start 2.05 -0.3)
-			(end 2.05 0.3)
+		(fp_arc
+			(start 1.35 -1)
+			(mid 1.844975 -0.794975)
+			(end 2.05 -0.3)
 			(stroke
 				(width 0.12)
@@
 		)
 		(fp_arc
+			(start 2.05 0.3)
+			(mid 1.844975 0.794975)
+			(end 1.35 1)
+			(stroke
+				(width 0.12)
+				(type solid)
+			)
+			(layer "F.SilkS")
+		)
+		(fp_arc
 			(start -1.35 1)
 			(mid -1.844975 0.794975)
@@
 			(layer "F.SilkS")
 		)
-		(fp_arc
-			(start 1.35 -1)
-			(mid 1.844975 -0.794975)
-			(end 2.05 -0.3)
-			(stroke
-				(width 0.12)
-				(type solid)
-			)
-			(layer "F.SilkS")
-		)
-		(fp_arc
-			(start 2.05 0.3)
-			(mid 1.844975 0.794975)
-			(end 1.35 1)
-			(stroke
-				(width 0.12)
-				(type solid)
-			)
-			(layer "F.SilkS")
+		(fp_line
+			(start -2.3 -1.25)
+			(end 2.3 -1.25)
+			(stroke
+				(width 0.05)
+				(type solid)
+			)
+			(layer "F.CrtYd")
 		)
 		(fp_line
@@
 		)
 		(fp_line
-			(start -2.3 -1.25)
+			(start 2.3 1.25)
 			(end 2.3 -1.25)
 			(stroke
@@
 			(layer "F.CrtYd")
 		)
-		(fp_line
-			(start 2.3 1.25)
-			(end 2.3 -1.25)
-			(stroke
-				(width 0.05)
-				(type solid)
-			)
-			(layer "F.CrtYd")
-		)
 		(pad "1" smd custom
-			(at -1.3 0)
+			(at -1.3 0 90)
 			(size 1 0.5)
 			(layers "F.Cu" "F.Mask")
@@
 		)
 		(pad "2" smd rect
-			(at 0 0)
+			(at 0 0 90)
 			(size 1 1.5)
 			(layers "F.Cu" "F.Mask")
@@
 		)
 		(pad "3" smd custom
-			(at 1.3 0)
+			(at 1.3 0 90)
 			(size 1 0.5)
 			(layers "F.Cu" "F.Mask")
-			(net "/5V")
+			(net "/5V_REG")
 			(zone_connect 2)
 			(thermal_bridge_angle 45)
@@
 			(layers "F.Cu" "F.Mask" "F.Paste")
 			(roundrect_rratio 0.25)
-			(net "/5V")
+			(net "/5V_REG")
 		)
 		(pad "2" smd roundrect
@@
 		(descr "14-lead though-hole mounted DIP package, row spacing 7.62mm (300 mils)")
 		(tags "THT DIP DIL PDIP 2.54mm 7.62mm 300mil")
-		(property "Reference" "U1"
+		(property "Reference" "U3"
 			(at 3.81 -2.33 0)
 			(layer "F.SilkS")
@@
 			(layers "*.Cu" "*.Mask")
 			(remove_unused_layers no)
-			(net "unconnected-(U1-Pad6)")
+			(net "unconnected-(U3-Pad6)")
 		)
 		(pad "7" thru_hole circle
@@
 			(layers "*.Cu" "*.Mask")
 			(remove_unused_layers no)
-			(net "unconnected-(U1-Pad8)")
+			(net "unconnected-(U3-Pad8)")
 		)
 		(pad "9" thru_hole circle
@@
 			(layers "*.Cu" "*.Mask")
 			(remove_unused_layers no)
-			(net "unconnected-(U1-Pad11)")
+			(net "unconnected-(U3-Pad11)")
 		)
 		(pad "12" thru_hole circle
@@
 			(layers "*.Cu" "*.Mask")
 			(remove_unused_layers no)
-			(net "/5V")
+			(net "/5V_REG")
 		)
 		(embedded_fonts no)
@@
 		(start 20.62 3)
 		(end 23.05 3)
-		(width 0.5)
-		(layer "F.Cu")
-		(net "/5V")
+		(width 1.5)
+		(layer "F.Cu")
+		(net "/5V_REG")
 	)
 	(segment
 		(start 5 5)
 		(end 5 3)
-		(width 0.5)
-		(layer "F.Cu")
-		(net "/5V")
+		(width 1.5)
+		(layer "F.Cu")
+		(net "/5V_REG")
 	)
 	(segment
 		(start 20.62 3)
 		(end 20.62 7.54)
-		(width 0.5)
-		(layer "F.Cu")
-		(net "/5V")
+		(width 1.5)
+		(layer "F.Cu")
+		(net "/5V_REG")
 	)
 	(segment
 		(start 5 3)
 		(end 20.62 3)
-		(width 0.5)
-		(layer "F.Cu")
-		(net "/5V")
+		(width 1.5)
+		(layer "F.Cu")
+		(net "/5V_REG")
 	)
 	(segment
-		(start 10.9 5.5)
-		(end 10.9 3)
-		(width 0.5)
-		(layer "F.Cu")
-		(net "/5V")
+		(start 9.6 3)
+		(end 9.6 3.9)
+		(width 1.5)
+		(layer "F.Cu")
+		(net "/5V_REG")
 	)
 	(segment
@@
 	)
 	(segment
-		(start 8.3 5.5)
-		(end 8.3 7.4)
+		(start 9.6 6.8)
+		(end 9.6 8.5)
 		(width 0.25)
 		(layer "F.Cu")
@@
 	)
 	(via
-		(at 8.3 7.4)
+		(at 9.6 8.5)
 		(size 0.8)
 		(drill 0.4)
@@
 	(segment
 		(start 9.6 5.5)
-		(end 9.6 7.54)
+		(end 11 5.5)
 		(width 0.25)
 		(layer "F.Cu")
@@
 	)
 	(segment
-		(start 9.6 7.54)
+		(start 11 5.5)
 		(end 13 7.54)
 		(width 0.25)
