Commit message: URDF e MJCF rigenerati sul cad.json del blocco A (massa 2950,7 g); 57 test Python e app verificati dopo l'unione

File: robot/generati/esapode.urdf (robot description, URDF)
Before this commit: robot esapode, 26 links, 25 joints
Links:
- link tibia_AD: mass 0.11019 -> 0.11144
- link tibia_AS: mass 0.11019 -> 0.11144
- link tibia_MD: mass 0.11019 -> 0.11144
- link tibia_MS: mass 0.11019 -> 0.11144
- link tibia_PD: mass 0.11019 -> 0.11144
- link tibia_PS: mass 0.11019 -> 0.11144

Commit message: 2.1.0 blocco B (D-066): 2813 fra SSC-32 e portafusibile, IMU e ADC sotto il vassoio, prese dei piedi, spie dei rail, ToF frontale con finestra e tappo, ToF posteriore, supporti degli INA260, anello del pulsante con camera nera, luci dei lobi, ganci, zaino, microfoni, altoparlante, ampli e scheda del carapace, FSR nella zampa; unioni limitate ai corpi della parte; descrizione del robot e file generati aggiornati

File: robot/generati/esapode.urdf (robot description, URDF)
Before this commit: robot esapode, 26 links, 25 joints
Links:
- link corpo: mass 1.39104 -> 1.42318
- link tibia_AD: mass 0.11144 -> 0.11174
- link tibia_AS: mass 0.11144 -> 0.11174
- link tibia_MD: mass 0.11144 -> 0.11174
- link tibia_MS: mass 0.11144 -> 0.11174
- link tibia_PD: mass 0.11144 -> 0.11174
- link tibia_PS: mass 0.11144 -> 0.11174

Commit message: 2.1.1: modelli URDF e MJCF rigenerati dalla descrizione (la CI sim li trovava vecchi); in CLAUDE.md la procedura elenca tutti i generatori

File: robot/generati/esapode.urdf (robot description, URDF)
Before this commit: robot esapode, 26 links, 25 joints
Links:
- link corpo: mass 1.42318 -> 1.42471
- link tibia_AD: mass 0.11174 -> 0.11189
- link tibia_AS: mass 0.11174 -> 0.11189
- link tibia_MD: mass 0.11174 -> 0.11189
- link tibia_MS: mass 0.11174 -> 0.11189
- link tibia_PD: mass 0.11174 -> 0.11189
- link tibia_PS: mass 0.11174 -> 0.11189

Commit message: Versione 2.1.2 (D-069): predisposizioni scelte (approvate e backlog), prese delle luci delle tibie, provino di luce, presa del T-plug verificata, tocco dai sensori esistenti in software.md; BOM con la sezione X divisa fra approvate e backlog

File: robot/generati/esapode.urdf (robot description, URDF)
Before this commit: robot esapode, 26 links, 25 joints
Links:
- link corpo: mass 1.42471 -> 1.42791

Commit message: Versione 2.1.3 (D-070): lame del femore come il guscio della tibia, chiuse su teste e mozzi, con la feritoia a intarsio nero; nessuna copertura superiore
- zampa.py: lame nuove (sagoma da X 40 a 135,5 con tre angoli smussati, faccia piana con smusso 3 x 2, tasche cieche per le 12 teste M3 sulla A e per i perni sulla B), intarsi Cover_Femore_A/B_Feritoia stampati con la lama; tolti i parametri delle lame bombate
- verifiche in CAD: zampa libera (81 pose, 17 controlli su 20), coxe a +-35, vicine libere a 30,5 e a contatto a 31 (gioco a 30 di 3,58 mm), carapace a 3,96 mm, cicli e rotazione liberi
- massa attesa 3060,6 g (femore al 53 % dello stallo): calc, robot.yaml, regressioni e test del contatto fra vicine aggiornati
- STL, esportazione del robot, generati, mesh e render delle zampe rifatti

File: robot/generati/esapode.urdf (robot description, URDF)
Before this commit: robot esapode, 26 links, 25 joints
Links:
- link femore_AD: mass 0.05442 -> 0.06615
- link femore_AS: mass 0.05442 -> 0.06615
- link femore_MD: mass 0.05442 -> 0.06615
- link femore_MS: mass 0.05442 -> 0.06615
- link femore_PD: mass 0.05442 -> 0.06615
- link femore_PS: mass 0.05442 -> 0.06615

Commit message: Versione 2.1.4 (D-071): lame del femore con la sagoma del femore e l'estetica della 2.1.3, feritoia al centro
- zampa.py: sagoma come le lame di D-061 (fascia a Z +-14,5, teste esagonali, rialzo da X 80 a 97 con rampe a 30 e 45 gradi), spigoli vivi con lo smusso 3 x 2; feritoia e viti della lama B a Z 1,5, vite lato ginocchio a X 89 (inserto di Femore_B spostato con la quota dello schizzo)
- verifiche in CAD: zampa libera, coxe a +-35, vicine libere a 30,5 e a contatto a 31, carapace a 4,58 mm, cicli e rotazione liberi
- massa attesa 3043,5 g (femore al 53 % dello stallo); STL, robot, generati, mesh e render aggiornati

File: robot/generati/esapode.urdf (robot description, URDF)
Before this commit: robot esapode, 26 links, 25 joints
Links:
- link femore_AD: mass 0.06615 -> 0.0633
- link femore_AS: mass 0.06615 -> 0.0633
- link femore_MD: mass 0.06615 -> 0.0633
- link femore_MS: mass 0.06615 -> 0.0633
- link femore_PD: mass 0.06615 -> 0.0633
- link femore_PS: mass 0.06615 -> 0.0633

Commit message: Versione 2.1.6 (D-074): doppia predisposizione di IMU (GY-6500 su Corpo_Piastrina_IMU sopra le bugne della Pololu) e microfoni (MS3625 centrate da Corpo_Lunette_Microfoni nella sede della Adafruit), amplificatore generico con le bugne sul lato della morsettiera (quelle in diagonale erano sbagliate), altoparlante tondo da 15 con fermo; controllo delle varianti con caso di controllo; massa attesa 3045,0 g; carapace a 3,96 mm dalle zampe medie (il 4,58 di D-071 non si ritrova); pull-down da 100 kΩ sui dati dei microfoni; BOM X4, X16, X17 in casa; verificato da tre revisori

File: robot/generati/esapode.urdf (robot description, URDF)
Before this commit: robot esapode, 26 links, 25 joints
Links:
- link corpo: mass 1.42791 -> 1.42943

Commit message: Versione 2.1.7, blocco a valle: STL, mesh, cad.json, pose e generatori rifatti dal modello, massa attesa 3047,2 g con la regressione, dati della guida (manifest, fori, catalogo e passi dei totali) allineati al vassoio sulle colonne, BOM e documenti della 2.1.7 con gli esiti nel piano

File: robot/generati/esapode.urdf (robot description, URDF)
Before this commit: robot esapode, 26 links, 25 joints
Links:
- link corpo: mass 1.42943 -> 1.43155

Commit message: Versione 2.1.7, correzioni della verifica: asola e ala del vassoio a x 30 fuori dalle prese dei piedi (Qwiic nella presa di coda dell'ADC), scheda del carapace alzata di 0,6 con inserti da 3,4 e viti M2 x 4, percorso del cavo piatto in due strisce, rebbi fino a z -19,9 per i cavi del pacco, pacco da 139,65 con la schiuma, lamatura dei LED delle spie fuori da F1, colonne del vassoio Ø6,6, carapace rifatto (raccordi persi dal ricalcolo); verifiche con scatole provvisorie e casi di controllo, massa attesa 3046,2 g, STL, mesh, cad.json, generatori e dati della guida; documenti, BOM, nota in D-071, scelta di P-015 in software.md, guida 8.07, 8.09, 11.03, 15.10, 15.11, lezioni del connettore

File: robot/generati/esapode.urdf (robot description, URDF)
Before this commit: robot esapode, 26 links, 25 joints
Links:
- link corpo: mass 1.43155 -> 1.43059

Commit message: 2.1.8, blocco E: a valle (STL, mesh, descrizione del robot e generati, massa attesa 3048,2 g, guida con la scheda dei partitori al passo 8.10 e le prese delle luci al 7.10, catalogo, BOM); contorno della PCB-P in genera_contorni

File: robot/generati/esapode.urdf (robot description, URDF)
Before this commit: robot esapode, 26 links, 25 joints
Links:
- link corpo: mass 1.43059 -> 1.43255
