File: pcb/basetta/basetta.kicad_sch (KiCad schematic)
At the start: 50 parts, among them P1 batteria (2813), P10 cavo piatto, P11 uscita di X3, P12 impulso RMT dalla SSC-32, P2 2813, P3 abilitazione (D2 in linea), P4 seriale SSC-32, P5 bus GND, P6 bus 3V3, P7 bus SDA, P8 bus SCL, P9 luci delle tibie, U1 ESP32-S3-CAM RE1.3, U2 D24V22F5, U3 SN74AHCT125N

Commit message: D-079: arresto R1 dei PCB approvato; correzioni della verifica con due agenti (TCA9534 tolto, R16 su OFF, regole del DRC per 5V/3V3 del carapace, EN di U2 e pulsante, testata con fori da 1,1, CS su due passi, tetto dei LED a 450 mA con l'audio)
Parts:
- added R16: 10k, hex2:R_Axial_DIN0207_L6.3mm_D2.5mm_P7.62mm_Horizontal, symbol hex2_kicad:R
- CS1, CS2: footprint hex2:C_Disc_D3.8mm_W2.6mm_P2.50mm -> hex2:C_Rect_L7.0mm_W3.5mm_P2.50mm_P5.00mm
Connections:
- net OFF: now also R16.1; no longer P2.2 (Pin_2)
- new net OFF_2813: P2.2 (Pin_2), R16.2
Other:
- moved on the sheet: R10, R11, R12, R13, R14, R15

Commit message: D-082: correzioni della revisione indipendente (17 agenti): PCB-C rifatta e sbrogliata da script (DRC a zero), regole del DRC corrette (una scritta male faceva ignorare il file), piazzole dei fili in verifica_reti, ali da 5,5, JP-RMT 680/1k, tetto dei LED 600/400 mA, guida 8.10/8.22/8.24, CI con KiCad obbligatorio; proposta della 2.1.9 (scheda dei partitori piu' grande)
Parts:
- R14: value 20k -> 680
- R15: value 33k -> 1k
Changed lines of the file:
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@@
 			)
 		)
-		(property "Value" "20k"
+		(property "Value" "680"
 			(at 340.36 142.24 90)
 			(show_name no)
@@
 			)
 		)
-		(property "Value" "33k"
+		(property "Value" "1k"
 			(at 360.68 142.24 90)
 			(show_name no)

Commit message: PCB-B, F4 (in corso): piazzamento da script con l'apertura sotto U2, VBAT da sotto accanto al VIN, varchi 23/27/28/30 sulla fila -Y, resistenze in piedi e 0805 sotto, PTC MF-R090-0-9, tolti JP-RMT e 11 punti di prova; DRC di piazzamento a zero; ingombri provati nel CAD (assieme.py -> basetta_pcb, nessun urto, 7 casi di controllo); dima, render e stampa 1:1 della basetta
Parts:
- removed JP2: JP-RMT, hex2:SolderJumper-2_P1.3mm_Open_RoundedPad1.0x1.5mm, symbol hex2_kicad:SolderJumper_2_Open
- removed P12: impulso RMT dalla SSC-32, hex2:PinHeader_1x02_P2.54mm_Vertical, symbol hex2_kicad:Conn_01x02
- removed R14: 680, hex2:R_Axial_DIN0207_L6.3mm_D2.5mm_P7.62mm_Horizontal, symbol hex2_kicad:R
- removed R15: 1k, hex2:R_Axial_DIN0207_L6.3mm_D2.5mm_P7.62mm_Horizontal, symbol hex2_kicad:R
- removed TP1: VBAT, hex2:TestPoint_THTPad_1.5x1.5mm_Drill0.7mm, symbol hex2_kicad:TestPoint
- removed TP10: SENSE, hex2:TestPoint_THTPad_1.5x1.5mm_Drill0.7mm, symbol hex2_kicad:TestPoint
- removed TP11: GPIO42, hex2:TestPoint_THTPad_1.5x1.5mm_Drill0.7mm, symbol hex2_kicad:TestPoint
- removed TP14: TX5, hex2:TestPoint_THTPad_1.5x1.5mm_Drill0.7mm, symbol hex2_kicad:TestPoint
- removed TP15: DATA, hex2:TestPoint_THTPad_1.5x1.5mm_Drill0.7mm, symbol hex2_kicad:TestPoint
- removed TP16: DATA_TIBIE, hex2:TestPoint_THTPad_1.5x1.5mm_Drill0.7mm, symbol hex2_kicad:TestPoint
- removed TP17: GND, hex2:TestPoint_THTPad_1.5x1.5mm_Drill0.7mm, symbol hex2_kicad:TestPoint
- removed TP3: 5V_LED, hex2:TestPoint_THTPad_1.5x1.5mm_Drill0.7mm, symbol hex2_kicad:TestPoint
- removed TP5: 3V3S, hex2:TestPoint_THTPad_1.5x1.5mm_Drill0.7mm, symbol hex2_kicad:TestPoint
- removed TP6: SDA, hex2:TestPoint_THTPad_1.5x1.5mm_Drill0.7mm, symbol hex2_kicad:TestPoint
- removed TP7: SCL, hex2:TestPoint_THTPad_1.5x1.5mm_Drill0.7mm, symbol hex2_kicad:TestPoint
- CS1, CS2: footprint hex2:C_Rect_L7.0mm_W3.5mm_P2.50mm_P5.00mm -> hex2:C_0805_2012Metric
- P1: footprint hex2:PinHeader_1x02_P2.54mm_Vertical -> hex2:Fili_1x02_P2.54mm_D1.7
- P10: footprint hex2:PinHeader_1x14_P2.54mm_Vertical -> hex2:Fili_1x14_P2.54mm_D1.7
- P11: footprint hex2:PinHeader_1x02_P2.54mm_Vertical -> hex2:Fili_1x01_P2.54mm_D1.5; symbol hex2_kicad:Conn_01x02 -> hex2_kicad:Conn_01x01
- P2: footprint hex2:PinHeader_1x02_P2.54mm_Vertical -> hex2:Fili_1x02_P2.54mm_D1.5
- P3: footprint hex2:PinHeader_1x01_P2.54mm_Vertical -> hex2:Fili_1x01_P2.54mm_D1.5
- P4: footprint hex2:PinHeader_1x03_P2.54mm_Vertical -> hex2:Fili_1x03_P2.54mm_D1.5
- P5, P6, P7, P8: footprint hex2:PinHeader_1x05_P2.54mm_Vertical -> hex2:Fili_1x05_P2.54mm_D1.5
- P9: value luci delle tibie -> dato delle luci delle tibie; footprint hex2:PinHeader_1x03_P2.54mm_Vertical -> hex2:Fili_1x01_P2.54mm_D1.5; symbol hex2_kicad:Conn_01x03 -> hex2_kicad:Conn_01x01
- PTC1: value MF-R090 -> MF-R090-0-9; footprint hex2:Fuse_Bourns_MF-R090_Sdraiato -> hex2:Fuse_Bourns_MF-R090-0-9_Sdraiato
- R1, R10, R16: footprint hex2:R_Axial_DIN0207_L6.3mm_D2.5mm_P7.62mm_Horizontal -> hex2:R_0805_2012Metric
- R13, R2, R4, R5, R7, R9: footprint hex2:R_Axial_DIN0207_L6.3mm_D2.5mm_P7.62mm_Horizontal -> hex2:R_Axial_DIN0207_L6.3mm_D2.5mm_P2.54mm_Vertical
Connections:
- net 5V_LED: now also PTC1.1; no longer P9.1 (Pin_1), PTC1.2
- net 5V_REG: now also PTC1.2; no longer PTC1.1
- net DATA_TIBIE: now also P9.1 (Pin_1); no longer P9.2 (Pin_2)
- net GND: no longer P11.2 (Pin_2), P9.3 (Pin_3)
- no-connect marks 29 -> 25
Other:
- moved on the sheet: R16, TP12, TP13, TP2, TP4, TP8, TP9

Commit message: D-083: dima della PCB-C; PCB-B piazzata e sbrogliata a quattro strati (scelta dell'utente) con DRC a zero: instradatore del progetto (script/sbroglio.py) per le reti con regole a coppie, Freerouting 2.5.0 per le altre, rifinitura; PTC MF-R090-0-9, 0805 sotto, resistenze in piedi, varchi 27/28/30/40, polo 14 tagliato, 3V3 a 0,3; ingombri nel CAD senza urti; dima e stampe
Parts:
- P10: footprint hex2:Fili_1x14_P2.54mm_D1.7 -> hex2:Fili_1x13_P2.54mm_D1.7; symbol hex2_kicad:Conn_01x14 -> hex2_kicad:Conn_01x13
Connections:
- no-connect marks 25 -> 24
Changed lines of the file:
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@@
 	)
 	(no_connect
-		(at 114.3 92.71)
+		(at 114.3 95.25)
 	)
 	(no_connect
@@
 	)
 	(no_connect
-		(at 114.3 113.03)
+		(at 114.3 115.57)
 	)
 	(no_connect
@@
 	)
 	(no_connect
-		(at 236.22 228.6)
+		(at 181.61 50.8)
 	)
 	(no_connect
-		(at 181.61 50.8)
+		(at 114.3 82.55)
 	)
 	(no_connect
@@
 	)
 	(no_connect
-		(at 114.3 90.17)
+		(at 114.3 92.71)
 	)
 	(no_connect
@@
 	)
 	(no_connect
-		(at 114.3 115.57)
-	)
-	(no_connect
 		(at 88.9 120.65)
 	)
@@
 	(wire
 		(pts
-			(xy 114.3 97.79) (xy 116.84 97.79)
+			(xy 114.3 100.33) (xy 116.84 100.33)
 		)
 		(stroke
@@
 	(wire
 		(pts
-			(xy 114.3 102.87) (xy 116.84 102.87)
+			(xy 114.3 105.41) (xy 116.84 105.41)
 		)
 		(stroke
@@
 	(wire
 		(pts
-			(xy 114.3 107.95) (xy 116.84 107.95)
+			(xy 114.3 110.49) (xy 116.84 110.49)
 		)
 		(stroke
@@
 	(wire
 		(pts
-			(xy 114.3 95.25) (xy 116.84 95.25)
+			(xy 114.3 97.79) (xy 116.84 97.79)
 		)
 		(stroke
@@
 	(wire
 		(pts
-			(xy 114.3 82.55) (xy 116.84 82.55)
+			(xy 114.3 85.09) (xy 116.84 85.09)
 		)
 		(stroke
@@
 	(wire
 		(pts
-			(xy 114.3 87.63) (xy 116.84 87.63)
+			(xy 114.3 90.17) (xy 116.84 90.17)
 		)
 		(stroke
@@
 	(wire
 		(pts
-			(xy 114.3 85.09) (xy 116.84 85.09)
+			(xy 114.3 87.63) (xy 116.84 87.63)
 		)
 		(stroke
@@
 	(wire
 		(pts
-			(xy 114.3 110.49) (xy 116.84 110.49)
+			(xy 114.3 113.03) (xy 116.84 113.03)
 		)
 		(stroke
@@
 	(wire
 		(pts
-			(xy 114.3 100.33) (xy 116.84 100.33)
+			(xy 114.3 102.87) (xy 116.84 102.87)
 		)
 		(stroke
@@
 	(wire
 		(pts
-			(xy 114.3 105.41) (xy 116.84 105.41)
+			(xy 114.3 107.95) (xy 116.84 107.95)
 		)
 		(stroke
@@
 	)
 	(label "LED_IN"
-		(at 116.84 87.63 0)
+		(at 116.84 90.17 0)
 		(effects
 			(font
@@
 	)
 	(label "BCLK"
-		(at 116.84 95.25 0)
+		(at 116.84 97.79 0)
 		(effects
 			(font
@@
 	)
 	(label "AMP"
-		(at 116.84 107.95 0)
+		(at 116.84 110.49 0)
 		(effects
 			(font
@@
 	)
 	(label "SENSE"
-		(at 116.84 110.49 0)
+		(at 116.84 113.03 0)
 		(effects
 			(font
@@
 	)
 	(label "MIC"
-		(at 116.84 100.33 0)
+		(at 116.84 102.87 0)
 		(effects
 			(font
@@
 	)
 	(label "TX3"
-		(at 116.84 82.55 0)
+		(at 116.84 85.09 0)
 		(effects
 			(font
@@
 	)
 	(label "SDA"
-		(at 116.84 85.09 0)
+		(at 116.84 87.63 0)
 		(effects
 			(font
@@
 	)
 	(label "WS"
-		(at 116.84 97.79 0)
+		(at 116.84 100.33 0)
 		(effects
 			(font
@@
 	)
 	(label "OFF"
-		(at 116.84 102.87 0)
+		(at 116.84 105.41 0)
 		(effects
 			(font
@@
 	)
 	(label "GPIO42"
-		(at 116.84 105.41 0)
+		(at 116.84 107.95 0)
 		(effects
 			(font
@@
 	)
 	(symbol
-		(lib_id "hex2_kicad:Conn_01x14")
+		(lib_id "hex2_kicad:Conn_01x13")
 		(at 241.3 210.82 0)
 		(unit 1)
@@
 		)
 		(property "Value" "cavo piatto"
-			(at 241.3 231.14 0)
+			(at 241.3 228.6 0)
 			(show_name no)
 			(do_not_autoplace no)
@@
 			)
 		)
-		(property "Footprint" "hex2:Fili_1x14_P2.54mm_D1.7"
+		(property "Footprint" "hex2:Fili_1x13_P2.54mm_D1.7"
 			(at 241.3 210.82 0)
 			(hide yes)
@@
 			)
 		)
-		(property "Description" "Generic connector, single row, 01x14, script generated (kicad-library-utils/schlib/autogen/connector/)"
+		(property "Description" "Generic connector, single row, 01x13, script generated (kicad-library-utils/schlib/autogen/connector/)"
 			(at 241.3 210.82 0)
 			(hide yes)
@@
 		(pin "13"
 		)
-		(pin "14"
-		)
 		(instances
 			(project "basetta"
@@
 		(pin "22"
 		)
+		(pin "23"
+		)
 		(pin "24"
 		)
@@
 		(pin "39"
 		)
-		(pin "40"
-		)
 		(instances
