File: pcb/partitori/partitori.kicad_pcb (KiCad board)
At the start: 4 copper layers, 33.8 x 8.6 mm, 18 parts, among them J1 pettine dei piedi, P1 NTC e ADC

Commit message: Versione 2.1.9 (D-085): scheda dei partitori nuova nel CAD e in KiCad con il contorno dal CAD, file Fusion versione 23; a valle (STL, mesh, descrizione del robot, guida 8.10 e 8.24); storico, decisione e stato
Other:
- outline, holes or cut-outs redrawn
